Commit message: added new dae file for skyrover nano and a launch file for ps4 controller

File: crazyflie_description/urdf/crazyflie.urdf.xacro (robot description, xacro)
@@ -1,5 +1,5 @@
 <?xml version="1.0"?>
 <robot xmlns:xacro="http://www.ros.org/wiki/xacro" name="crazyflie">
-  <link name="base_link">
+  <link name="/crazyflie/base_link">
     <inertial>
       <mass value="0.019" />
@@ -11,5 +11,5 @@
       <origin xyz="0 0 0" rpy="0 0 0" />
       <geometry>
-        <mesh filename="package://crazyflie_description/meshes/crazyflie.dae"/>
+        <mesh filename="package://crazyflie_description/meshes/skyrover_nano_v2.dae"/>
       </geometry>
     </visual>
